File: max_breakout.sch (KiCad schematic (older format))
At the start: 55 parts, among them J1 Right, J2 Left, J3 AVR-JTAG-10, J4 USB_B_Micro, Q1 IRLML6402, SW1 User DIP Switch, SW2 Reset, SW3 Reset, U1 AP7381-33SA, U2 EPM7032STC44, U3 MAX40200AUK, U4 MAX40200AUK, U5 74HCT365, U6 74HCT2G125, U7 DS1813R-5+T&R, X1 CTX-636 50mhz

Commit message: docs, images and gerbers
Connections:
- wire segments 238 -> 239
Other:
- moved on the sheet: JP2, R18
Changed lines of the file:
@@
-$EndComp
-$Comp
-L Device:LED_Dual_ACAC D3
-U 1 1 5D298EB6
-P 4804 6385
-F 0 "D3" H 4804 6038 50  0000 C CNN
-F 1 "LED" H 4804 6129 50  0000 C CNN
-F 2 "LED_SMD:LED_2C_0603_1608Metric_Pad1.05x0.95mm_HandSolder" H 4834 6385 50  0001 C CNN
-F 3 "https://www.mouser.com/datasheet/2/348/sml-d22-e-1508165.pdf" H 4834 6385 50  0001 C CNN
-F 4 "Standard LEDs - SMD Red/YelGrn 620/570nm 16/10mcd 65/67mW 5mA" H 4804 6385 50  0001 C CNN "Description"
-F 5 "SML-D22MUWT86" H 4804 6385 50  0001 C CNN "MPN"
-F 6 "ROHM Semiconductor" H 4804 6385 50  0001 C CNN "Manufacturer"
-	1    4804 6385
-	1    0    0    -1
 $EndComp
 $Comp
@@
 Text Label 5529 6940 1    50   ~ 0
 LED_ENA
-$Comp
-L Device:R_Small R17
-U 1 1 5D298EC1
-P 4404 6285
-F 0 "R17" V 4439 6430 50  0000 C CNN
-F 1 "360R" V 4402 6289 32  0000 C CNN
-F 2 "Resistor_SMD:R_0603_1608Metric_Pad1.05x0.95mm_HandSolder" H 4404 6285 50  0001 C CNN
-F 3 "https://www.mouser.com/datasheet/2/54/hpreztr-777398.pdf" H 4404 6285 50  0001 C CNN
-F 4 "Thick Film Resistors - SMD 10K 1% 1/10W" H 4404 6285 50  0001 C CNN "Description"
-F 5 "CR0603-FX-1002ELF" H 4404 6285 50  0001 C CNN "MPN"
-F 6 "Bourns" H 4404 6285 50  0001 C CNN "Manufacturer"
-	1    4404 6285
-	0    1    -1   0
-$EndComp
-$Comp
-L Device:R_Small R19
-U 1 1 5D4B3D04
-P 4404 6485
-F 0 "R19" V 4438 6628 50  0000 C CNN
-F 1 "360R" V 4406 6485 32  0000 C CNN
-F 2 "Resistor_SMD:R_0603_1608Metric_Pad1.05x0.95mm_HandSolder" H 4404 6485 50  0001 C CNN
-F 3 "https://www.mouser.com/datasheet/2/54/hpreztr-777398.pdf" H 4404 6485 50  0001 C CNN
-F 4 "Thick Film Resistors - SMD 10K 1% 1/10W" H 4404 6485 50  0001 C CNN "Description"
-F 5 "CR0603-FX-1002ELF" H 4404 6485 50  0001 C CNN "MPN"
-F 6 "Bourns" H 4404 6485 50  0001 C CNN "Manufacturer"
-	1    4404 6485
-	0    1    -1   0
-$EndComp
-$Comp
-L power:VCC #PWR032
-U 1 1 5D89D858
-P 4172 6388
-F 0 "#PWR032" H 4172 6238 50  0001 C CNN
-F 1 "VCC" H 4189 6561 50  0000 C CNN
-F 2 "" H 4172 6388 50  0001 C CNN
-F 3 "" H 4172 6388 50  0001 C CNN
-	1    4172 6388
-	0    -1   -1   0
-$EndComp
-Wire Wire Line
-	4304 6285 4304 6388
-Wire Wire Line
-	4304 6388 4172 6388
-Connection ~ 4304 6388
-Wire Wire Line
-	4304 6388 4304 6485
 Text Label 10000 900  0    50   ~ 0
 5V_in
@@
 Text Notes 750  4900 0    50   ~ 0
 USER GPIO
-$Comp
-L Jumper:Jumper_2_Open JP2
-U 1 1 5E298777
-P 1000 6800
-F 0 "JP2" H 1000 7024 50  0000 C CNN
-F 1 "SW_EN" H 1000 6933 50  0000 C CNN
-F 2 "Connector_PinHeader_1.27mm:PinHeader_1x02_P1.27mm_Vertical" H 1000 6800 50  0001 C CNN
-F 3 "~" H 1000 6800 50  0001 C CNN
-	1    1000 6800
-	0    -1   -1   0
-$EndComp
-$Comp
-L power:VCC #PWR030
-U 1 1 5E298783
-P 1000 6250
-F 0 "#PWR030" H 1000 6100 50  0001 C CNN
-F 1 "VCC" H 1017 6423 50  0000 C CNN
-F 2 "" H 1000 6250 50  0001 C CNN
-F 3 "" H 1000 6250 50  0001 C CNN
-	1    1000 6250
-	1    0    0    -1
-$EndComp
-$Comp
-L max_breakout-rescue:GND-power #PWR034
-U 1 1 5E298789
-P 1000 7000
-AR Path="/5E298789" Ref="#PWR034"  Part="1"
-AR Path="/5D0F9837/5E298789" Ref="#PWR?"  Part="1"
-AR Path="/5CFABACD/5E298789" Ref="#PWR?"  Part="1"
-AR Path="/5CFABACD/5CFFC458/5E298789" Ref="#PWR?"  Part="1"
-AR Path="/5D65A6A0/5E298789" Ref="#PWR?"  Part="1"
-F 0 "#PWR034" H 1000 6750 50  0001 C CNN
-F 1 "GND" H 1005 6827 50  0000 C CNN
-F 2 "" H 1000 7000 50  0001 C CNN
-F 3 "" H 1000 7000 50  0001 C CNN
-	1    1000 7000
-	1    0    0    -1
-$EndComp
 Wire Notes Line
 	595  690  3400 690
@@
 JTAG
 Wire Wire Line
-	5105 6285 5229 6285
-Connection ~ 5229 6285
-Wire Wire Line
 	5229 6285 5230 6285
 Wire Wire Line
-	5105 6485 5229 6485
-Connection ~ 5229 6485
-Wire Wire Line
 	5229 6485 5230 6485
-Connection ~ 5104 6285
-Connection ~ 5104 6485
 $Comp
 L max_breakout-rescue:GND-power #PWR024
@@
 Wire Wire Line
 	3300 4250 3500 4250
-Wire Wire Line
-	1000 6600 1550 6600
-$Comp
-L max_breakout-rescue:R_Small-Device R18
-U 1 1 5E29877D
-P 1000 6400
-F 0 "R18" H 1010 6260 50  0000 L CNN
-F 1 "10K" V 1000 6350 50  0000 L CNN
-F 2 "Resistor_SMD:R_0603_1608Metric_Pad1.05x0.95mm_HandSolder" H 1000 6400 50  0001 C CNN
-F 3 "~" H 1000 6400 50  0001 C CNN
-	1    1000 6400
-	-1   0    0    1
-$EndComp
-Wire Wire Line
-	1000 6500 1000 6600
-Connection ~ 1000 6600
 $Comp
 L max_breakout-rescue:R_Small-Device R?
@@
 Wire Wire Line
 	8850 4700 8850 4850
-Wire Wire Line
-	1000 6300 1000 6250
 Wire Wire Line
 	1300 5550 1300 5650
@@
 Text Label 2350 6300 0    50   ~ 0
 SW_ENA
-Text Label 1200 6600 0    50   ~ 0
+Text Label 2150 6800 0    50   ~ 0
 SW_ENA
 $Comp
@@
 Text Label 10000 1000 0    50   ~ 0
 CLK1
+$Comp
+L power:VCC #PWR032
+U 1 1 5D89D858
+P 4172 6388
+F 0 "#PWR032" H 4172 6238 50  0001 C CNN
+F 1 "VCC" H 4189 6561 50  0000 C CNN
+F 2 "" H 4172 6388 50  0001 C CNN
+F 3 "" H 4172 6388 50  0001 C CNN
+	1    4172 6388
+	0    -1   -1   0
+$EndComp
+$Comp
+L Device:R_Small R19
+U 1 1 5D4B3D04
+P 4404 6485
+F 0 "R19" V 4438 6628 50  0000 C CNN
+F 1 "360R" V 4406 6485 32  0000 C CNN
+F 2 "Resistor_SMD:R_0603_1608Metric_Pad1.05x0.95mm_HandSolder" H 4404 6485 50  0001 C CNN
+F 3 "https://www.mouser.com/datasheet/2/54/hpreztr-777398.pdf" H 4404 6485 50  0001 C CNN
+F 4 "Thick Film Resistors - SMD 10K 1% 1/10W" H 4404 6485 50  0001 C CNN "Description"
+F 5 "CR0603-FX-1002ELF" H 4404 6485 50  0001 C CNN "MPN"
+F 6 "Bourns" H 4404 6485 50  0001 C CNN "Manufacturer"
+	1    4404 6485
+	0    1    -1   0
+$EndComp
+$Comp
+L Device:R_Small R17
+U 1 1 5D298EC1
+P 4404 6285
+F 0 "R17" V 4439 6430 50  0000 C CNN
+F 1 "360R" V 4402 6289 32  0000 C CNN
+F 2 "Resistor_SMD:R_0603_1608Metric_Pad1.05x0.95mm_HandSolder" H 4404 6285 50  0001 C CNN
+F 3 "https://www.mouser.com/datasheet/2/54/hpreztr-777398.pdf" H 4404 6285 50  0001 C CNN
+F 4 "Thick Film Resistors - SMD 10K 1% 1/10W" H 4404 6285 50  0001 C CNN "Description"
+F 5 "CR0603-FX-1002ELF" H 4404 6285 50  0001 C CNN "MPN"
+F 6 "Bourns" H 4404 6285 50  0001 C CNN "Manufacturer"
+	1    4404 6285
+	0    1    -1   0
+$EndComp
+$Comp
+L Device:LED_Dual_ACAC D3
+U 1 1 5D298EB6
+P 4804 6385
+F 0 "D3" H 4804 6038 50  0000 C CNN
+F 1 "LED" H 4804 6129 50  0000 C CNN
+F 2 "LED_SMD:LED_2C_0603_1608Metric_Pad1.05x0.95mm_HandSolder" H 4834 6385 50  0001 C CNN
+F 3 "https://www.mouser.com/datasheet/2/348/sml-d22-e-1508165.pdf" H 4834 6385 50  0001 C CNN
+F 4 "Standard LEDs - SMD Red/YelGrn 620/570nm 16/10mcd 65/67mW 5mA" H 4804 6385 50  0001 C CNN "Description"
+F 5 "SML-D22MUWT86" H 4804 6385 50  0001 C CNN "MPN"
+F 6 "ROHM Semiconductor" H 4804 6385 50  0001 C CNN "Manufacturer"
+	1    4804 6385
+	1    0    0    -1
+$EndComp
+Connection ~ 4304 6388
+Wire Wire Line
+	4304 6388 4172 6388
+Wire Wire Line
+	4304 6285 4304 6388
+Wire Wire Line
+	4304 6388 4304 6485
+Connection ~ 5229 6485
+Connection ~ 5104 6485
+Wire Wire Line
+	5105 6485 5229 6485
+Connection ~ 5229 6285
+Connection ~ 5104 6285
+Wire Wire Line
+	5105 6285 5229 6285
+$Comp
+L max_breakout-rescue:R_Small-Device R18
+U 1 1 5E29877D
+P 1950 6650
+F 0 "R18" H 1960 6510 50  0000 L CNN
+F 1 "10K" V 1950 6600 50  0000 L CNN
+F 2 "Resistor_SMD:R_0603_1608Metric_Pad1.05x0.95mm_HandSolder" H 1950 6650 50  0001 C CNN
+F 3 "~" H 1950 6650 50  0001 C CNN
+	1    1950 6650
+	-1   0    0    1
+$EndComp
+$Comp
+L max_breakout-rescue:GND-power #PWR034
+U 1 1 5E298789
+P 1950 7250
+AR Path="/5E298789" Ref="#PWR034"  Part="1"
+AR Path="/5D0F9837/5E298789" Ref="#PWR?"  Part="1"
+AR Path="/5CFABACD/5E298789" Ref="#PWR?"  Part="1"
+AR Path="/5CFABACD/5CFFC458/5E298789" Ref="#PWR?"  Part="1"
+AR Path="/5D65A6A0/5E298789" Ref="#PWR?"  Part="1"
+F 0 "#PWR034" H 1950 7000 50  0001 C CNN
+F 1 "GND" H 1955 7077 50  0000 C CNN
+F 2 "" H 1950 7250 50  0001 C CNN
+F 3 "" H 1950 7250 50  0001 C CNN
+	1    1950 7250
+	1    0    0    -1
+$EndComp
+$Comp
+L power:VCC #PWR030
+U 1 1 5E298783
+P 1950 6500
+F 0 "#PWR030" H 1950 6350 50  0001 C CNN
+F 1 "VCC" H 1967 6673 50  0000 C CNN
+F 2 "" H 1950 6500 50  0001 C CNN
+F 3 "" H 1950 6500 50  0001 C CNN
+	1    1950 6500
+	1    0    0    -1
+$EndComp
+$Comp
+L Jumper:Jumper_2_Open JP2
+U 1 1 5E298777
+P 1950 7050
+F 0 "JP2" H 1950 7274 50  0000 C CNN
+F 1 "SW_EN" H 1950 7183 50  0000 C CNN
+F 2 "Connector_PinHeader_1.27mm:PinHeader_1x02_P1.27mm_Vertical" H 1950 7050 50  0001 C CNN
+F 3 "~" H 1950 7050 50  0001 C CNN
+	1    1950 7050
+	0    -1   -1   0
+$EndComp
+Wire Wire Line
+	1950 6550 1950 6500
+Wire Wire Line
+	1950 6750 1950 6800
+Wire Wire Line
+	1950 6800 2500 6800
+Connection ~ 1950 6800
+Wire Wire Line
+	1950 6800 1950 6850
 $EndSCHEMATC

Commit message: changed  layout
Parts:
- SW2: renamed from SW3; value Reset -> User
- U3: renamed from U7; symbol Power_Supervisor:DS1813R-5+T&R -> max_breakout-rescue:DS1813R-5+T&R-Power_Supervisor
- renumbered C13 to C12, C12 to C13, J2 to J1, J1 to J2, JP3 to JP1, JP1 to JP3, R19 to R18, R18 to R19, R9 to R20, R20 to R9, SW2 to SW1, SW1 to SW3, U3 to U4, U4 to U5, U5 to U6, U6 to U7
Other:
- moved on the sheet: D1, R6, SW1

Commit message: routed
Connections:
- wire segments 239 -> 237
Other:
- moved on the sheet: R17, R18
Changed lines of the file:
@@
 CLK1
-$Comp
-L power:VCC #PWR033
-U 1 1 5D89D858
-P 4172 6388
-F 0 "#PWR033" H 4172 6238 50  0001 C CNN
-F 1 "VCC" H 4189 6561 50  0000 C CNN
-F 2 "" H 4172 6388 50  0001 C CNN
-F 3 "" H 4172 6388 50  0001 C CNN
-	1    4172 6388
-	0    -1   -1   0
-$EndComp
 $Comp
 L Device:R_Small R18
 U 1 1 5D4B3D04
-P 4404 6485
-F 0 "R18" V 4438 6628 50  0000 C CNN
-F 1 "360R" V 4406 6485 32  0000 C CNN
-F 2 "Resistor_SMD:R_0603_1608Metric_Pad1.05x0.95mm_HandSolder" H 4404 6485 50  0001 C CNN
-F 3 "https://www.mouser.com/datasheet/2/54/hpreztr-777398.pdf" H 4404 6485 50  0001 C CNN
-F 4 "Thick Film Resistors - SMD 10K 1% 1/10W" H 4404 6485 50  0001 C CNN "Description"
-F 5 "CR0603-FX-1002ELF" H 4404 6485 50  0001 C CNN "MPN"
-F 6 "Bourns" H 4404 6485 50  0001 C CNN "Manufacturer"
-	1    4404 6485
+P 4529 6485
+F 0 "R18" V 4563 6628 50  0000 C CNN
+F 1 "360R" V 4531 6485 32  0000 C CNN
+F 2 "Resistor_SMD:R_0603_1608Metric_Pad1.05x0.95mm_HandSolder" H 4529 6485 50  0001 C CNN
+F 3 "https://www.mouser.com/datasheet/2/54/hpreztr-777398.pdf" H 4529 6485 50  0001 C CNN
+F 4 "Thick Film Resistors - SMD 10K 1% 1/10W" H 4529 6485 50  0001 C CNN "Description"
+F 5 "CR0603-FX-1002ELF" H 4529 6485 50  0001 C CNN "MPN"
+F 6 "Bourns" H 4529 6485 50  0001 C CNN "Manufacturer"
+	1    4529 6485
 	0    1    -1   0
 $EndComp
@@
 L Device:R_Small R17
 U 1 1 5D298EC1
-P 4404 6285
-F 0 "R17" V 4439 6430 50  0000 C CNN
-F 1 "360R" V 4402 6289 32  0000 C CNN
-F 2 "Resistor_SMD:R_0603_1608Metric_Pad1.05x0.95mm_HandSolder" H 4404 6285 50  0001 C CNN
-F 3 "https://www.mouser.com/datasheet/2/54/hpreztr-777398.pdf" H 4404 6285 50  0001 C CNN
-F 4 "Thick Film Resistors - SMD 10K 1% 1/10W" H 4404 6285 50  0001 C CNN "Description"
-F 5 "CR0603-FX-1002ELF" H 4404 6285 50  0001 C CNN "MPN"
-F 6 "Bourns" H 4404 6285 50  0001 C CNN "Manufacturer"
-	1    4404 6285
+P 4529 6285
+F 0 "R17" V 4564 6430 50  0000 C CNN
+F 1 "360R" V 4527 6289 32  0000 C CNN
+F 2 "Resistor_SMD:R_0603_1608Metric_Pad1.05x0.95mm_HandSolder" H 4529 6285 50  0001 C CNN
+F 3 "https://www.mouser.com/datasheet/2/54/hpreztr-777398.pdf" H 4529 6285 50  0001 C CNN
+F 4 "Thick Film Resistors - SMD 10K 1% 1/10W" H 4529 6285 50  0001 C CNN "Description"
+F 5 "CR0603-FX-1002ELF" H 4529 6285 50  0001 C CNN "MPN"
+F 6 "Bourns" H 4529 6285 50  0001 C CNN "Manufacturer"
+	1    4529 6285
 	0    1    -1   0
 $EndComp
-$Comp
-L Device:LED_Dual_ACAC D3
-U 1 1 5D298EB6
-P 4804 6385
-F 0 "D3" H 4804 6038 50  0000 C CNN
-F 1 "LED" H 4804 6129 50  0000 C CNN
-F 2 "LED_SMD:LED_2C_0603_1608Metric_Pad1.05x0.95mm_HandSolder" H 4834 6385 50  0001 C CNN
-F 3 "https://www.mouser.com/datasheet/2/348/sml-d22-e-1508165.pdf" H 4834 6385 50  0001 C CNN
-F 4 "Standard LEDs - SMD Red/YelGrn 620/570nm 16/10mcd 65/67mW 5mA" H 4804 6385 50  0001 C CNN "Description"
-F 5 "SML-D22MUWT86" H 4804 6385 50  0001 C CNN "MPN"
-F 6 "ROHM Semiconductor" H 4804 6385 50  0001 C CNN "Manufacturer"
-	1    4804 6385
-	1    0    0    -1
-$EndComp
-Connection ~ 4304 6388
+Connection ~ 4429 6388
 Wire Wire Line
-	4304 6388 4172 6388
+	4429 6285 4429 6388
 Wire Wire Line
-	4304 6285 4304 6388
-Wire Wire Line
-	4304 6388 4304 6485
-Connection ~ 5229 6485
-Connection ~ 5104 6485
-Wire Wire Line
-	5105 6485 5229 6485
-Connection ~ 5229 6285
-Connection ~ 5104 6285
-Wire Wire Line
-	5105 6285 5229 6285
+	4429 6388 4429 6485
 $Comp
 L max_breakout-rescue:R_Small-Device R19
@@
 Wire Wire Line
 	1950 6800 1950 6850
+$Comp
+L Device:LED_Dual_ACAC D3
+U 1 1 5D298EB6
+P 4929 6385
+F 0 "D3" H 4929 6038 50  0000 C CNN
+F 1 "LED" H 4929 6129 50  0000 C CNN
+F 2 "LED_SMD:LED_2C_0603_1608Metric_Pad1.05x0.95mm_HandSolder" H 4959 6385 50  0001 C CNN
+F 3 "https://www.mouser.com/datasheet/2/348/sml-d22-e-1508165.pdf" H 4959 6385 50  0001 C CNN
+F 4 "Standard LEDs - SMD Red/YelGrn 620/570nm 16/10mcd 65/67mW 5mA" H 4929 6385 50  0001 C CNN "Description"
+F 5 "SML-D22MUWT86" H 4929 6385 50  0001 C CNN "MPN"
+F 6 "ROHM Semiconductor" H 4929 6385 50  0001 C CNN "Manufacturer"
+	1    4929 6385
+	1    0    0    -1
+$EndComp
+Connection ~ 5229 6285
+Connection ~ 5229 6485
+Wire Wire Line
+	4429 6388 4297 6388
+$Comp
+L power:VCC #PWR033
+U 1 1 5D89D858
+P 4297 6388
+F 0 "#PWR033" H 4297 6238 50  0001 C CNN
+F 1 "VCC" H 4314 6561 50  0000 C CNN
+F 2 "" H 4297 6388 50  0001 C CNN
+F 3 "" H 4297 6388 50  0001 C CNN
+	1    4297 6388
+	0    -1   -1   0
+$EndComp
 $EndSCHEMATC

Commit message: version 1.1
Connections:
- net labels added: ~OE1
- net labels removed: OE1, ~USRPB
- wire segments 237 -> 238
Changed lines of the file:
@@
 ~RST
 Text Label 10000 1200 0    50   ~ 0
-OE1
+~OE1
 Text Label 10000 1500 0    50   ~ 0
 B18
@@
 L max_breakout-rescue:GND-power #PWR014
 U 1 1 5D403069
-P 7750 3550
+P 7750 3600
 AR Path="/5D403069" Ref="#PWR014"  Part="1"
 AR Path="/5CB63856/5D403069" Ref="#PWR?"  Part="1"
@@
 AR Path="/5CFABACD/5D403069" Ref="#PWR?"  Part="1"
 AR Path="/5CF9C1ED/5D403069" Ref="#PWR?"  Part="1"
-F 0 "#PWR014" H 7750 3300 50  0001 C CNN
-F 1 "GND" H 7750 3400 50  0000 C CNN
-F 2 "" H 7750 3550 50  0001 C CNN
-F 3 "" H 7750 3550 50  0001 C CNN
-	1    7750 3550
+F 0 "#PWR014" H 7750 3350 50  0001 C CNN
+F 1 "GND" H 7750 3450 50  0000 C CNN
+F 2 "" H 7750 3600 50  0001 C CNN
+F 3 "" H 7750 3600 50  0001 C CNN
+	1    7750 3600
 	1    0    0    -1
 $EndComp
@@
 ~RST
 Text Label 3900 3050 0    50   ~ 0
-~USRPB
+~OE1
 $Comp
 L max_breakout-rescue:EPM7032STC44-CPLD_Altera-sbc_z80-rescue U2
@@
 $EndComp
 Text Label 5400 5350 0    50   ~ 0
-~USRPB
+~OE1
 $Comp
 L power:VCC #PWR09
@@
 	0    -1   -1   0
 $EndComp
+Wire Wire Line
+	7750 3600 7750 3550
 $EndSCHEMATC

Commit message: fixed up gnd planes
Connections:
- net labels removed: SW_ENA
Other:
- moved on the sheet: C10, C11, C12, C13, C2, C3, C4, C5, C6, C7, C8, C9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

Commit message: fixed 3.3v reg pinouts, added thermal vias
Parts:
- D1: value Blue -> Red
- D3: symbol Device:LED_Dual_ACAC -> Device:LED_Bicolor
- J4: footprint Connector_USB:USB_Micro-B_Molex-105017-0001 -> Connector_USB:USB_Micro-B_Amphenol_10103594-0001LF_Horizontal
- R6: value 100R -> 360R
- U1: symbol Regulator_Linear:AP7381-33SA -> max_breakout-rescue:AP7381-33SA-Regulator_Linear
- U2: footprint Package_QFP:TQFP-44_10x10mm_P0.8mm -> Package_QFP:TQFP-44_10x10mm_P0.8mm_ThermalVias
Other:
- moved on the sheet: JP3, R17, R18, R20, U7A, U7B

Commit message: rerouted and updated BOM
Parts:
- removed C6: 100nF, Capacitor_SMD:C_0603_1608Metric_Pad1.05x0.95mm_HandSolder, symbol max_breakout-rescue:C_Small-Device
- removed D3: LED, LED_SMD:LED_2C_0603_1608Metric_Pad1.05x0.95mm_HandSolder, symbol Device:LED_Bicolor
- removed JP1: PB_EN, Connector_PinHeader_1.27mm:PinHeader_1x02_P1.27mm_Vertical, symbol Jumper:Jumper_2_Open
- removed JP2: SW_EN, Connector_PinHeader_1.27mm:PinHeader_1x02_P1.27mm_Vertical, symbol Jumper:Jumper_2_Open
- removed JP3: LED_EN, Connector_PinHeader_1.27mm:PinHeader_1x02_P1.27mm_Vertical, symbol Jumper:Jumper_2_Open
- removed R17: 360R, Resistor_SMD:R_0603_1608Metric_Pad1.05x0.95mm_HandSolder, symbol Device:R_Small
- removed R19, R20: 10K, Resistor_SMD:R_0603_1608Metric_Pad1.05x0.95mm_HandSolder, symbol max_breakout-rescue:R_Small-Device
- removed U6: 74HCT365, Package_SO:TSSOP-16_4.4x5mm_P0.65mm, symbol max_breakout-rescue:74HCT365-74xx
- removed U7: 74HCT2G125, Package_SO:TSSOP-8_3x3mm_P0.65mm, symbol max_breakout-rescue:74HCT2G125-74xGxx
- added D3: RGB, LED_SMD:IN-S85TATRGB, symbol Device:LED_RGAB
- added SW4: ENA Switch, Button_Switch_SMD:SW_DIP_SPSTx04_Slide_KingTek_DSHP04TS_W7.62mm_P1.27mm, symbol Switch:SW_DIP_x04
- added U6: 74HCT244, Package_SO:TSSOP-20_4.4x6.5mm_P0.65mm, symbol 74xx:74HCT244
- C1: Datasheet (none) -> https://www.mouser.com/datasheet/2/396/mlcc02_e-1307760.pdf; Description Multilayer Ceramic Capacitors MLCC - SMD/SMT 0603 6.3V 0.47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 -> Multilayer Ceramic Capacitors MLCC - SMD/SMT 0603 6.3V 2.2u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; Footprint (none) -> Capacitor_SMD:C_0603_1608Metric_Pad1.05x0.95mm_HandSolder; MFR Taiyo Yuden -> Murata; Value (none) -> 2.2uF
- C10, C8, C9: Datasheet (none) -> https://www.mouser.com/datasheet/2/396/mlcc02_e-1307760.pdf; Description Multilayer Ceramic Capacitors MLCC - SMD/SMT 0603 6.3V 0.47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 -> Multilayer Ceramic Capacitors MLCC - SMD/SMT 0603 6.3V 0.33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; Footprint (none) -> Capacitor_SMD:C_0603_1608Metric_Pad1.05x0.95mm_HandSolder; MFR Taiyo Yuden -> Murata; Value (none) -> .33uF
- C11: Datasheet (none) -> https://www.mouser.com/datasheet/2/396/mlcc02_e-1307760.pdf; Description Multilayer Ceramic Capacitors MLCC - SMD/SMT 0603 6.3V 0.47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 -> Multilayer Ceramic Capacitors MLCC - SMD/SMT 0603 6.3V 0..3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; Footprint (none) -> Capacitor_SMD:C_0603_1608Metric_Pad1.05x0.95mm_HandSolder; MFR Taiyo Yuden -> Murata; Value (none) -> .33uF
- C12, C2, C3, C4, C5, C7: Datasheet (none) -> https://www.mouser.com/datasheet/2/396/mlcc02_e-1307760.pdf; Description Multilayer Ceramic Capacitors MLCC - SMD/SMT 0603 6.3V 0.47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 -> Multilayer Ceramic Capacitors MLCC - SMD/SMT 0603 6.3V 100n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; Footprint (none) -> Capacitor_SMD:C_0603_1608Metric_Pad1.05x0.95mm_HandSolder; MFR Taiyo Yuden -> Murata; Value (none) -> 100nF
- C13: Datasheet (none) -> https://www.mouser.com/datasheet/2/396/mlcc02_e-1307760.pdf; Description Multilayer Ceramic Capacitors MLCC - SMD/SMT 0.1uF 25V X5R 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 -> Multilayer Ceramic Capacitors MLCC - SMD/SMT 0603 6.3V 100n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; Footprint (none) -> Capacitor_SMD:C_0603_1608Metric_Pad1.05x0.95mm_HandSolder; MFR Taiyo Yuden -> Murata; Value (none) -> 100nF
- D1: Datasheet (none) -> https://www.mouser.com/datasheet/2/216/APT1608EC-34957.pdf; Description (none) -> Standard LEDs - SMD RED WATER CLEAR; Footprint (none) -> LED_SMD:LED_0603_1608Metric_Pad1.05x0.95mm_HandSolder; MFR (none) -> Kingbright; MPN (none) -> APT1608EC; SPN (none) -> 604-APT1608EC; SPR (none) -> Mouser; SPURL (none) -> https://www.mouser.com/ProductDetail/604-APT1608EC; Value (none) -> Red
- D2: Datasheet (none) -> https://www.mouser.com/datasheet/2/216/APT1608SGC-32861.pdf; Description (none) -> Standard LEDs - SMD GREEN WATER CLEAR; Footprint (none) -> LED_SMD:LED_0603_1608Metric_Pad1.05x0.95mm_HandSolder; MFR (none) -> Kingbright; MPN (none) -> APT1608SGC; SPN (none) -> 604-APT1608SGC; SPR (none) -> Mouser; SPURL (none) -> https://www.mouser.com/ProductDetail/604-APT1608SGC; Value (none) -> Green
- J1: Footprint (none) -> Connector_PinHeader_2.54mm:PinHeader_1x19_P2.54mm_Vertical; Value (none) -> Left
- J2: Footprint (none) -> Connector_PinHeader_2.54mm:PinHeader_1x19_P2.54mm_Vertical; Value (none) -> Right
- J3: Footprint (none) -> Connector_PinHeader_2.54mm:PinHeader_2x05_P2.54mm_Vertical; Value (none) -> AVR-JTAG-10
- J4: Datasheet (none) -> https://www.mouser.com/datasheet/2/18/10103594-1361315.pdf; Description (none) -> USB Connectors 5P Quick Connect Micro USB TypeB Rcpt; Footprint (none) -> Connector_USB:USB_Micro-B_Amphenol_10103594-0001LF_Horizont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; MFR (none) -> Amphenol; MPN (none) -> 10103594-0001LF; SPN (none) -> 649-10103594-0001LF; SPR (none) -> Mouser; SPURL (none) -> https://www.mouser.com/ProductDetail/649-10103594-0001LF; Value (none) -> USB_B_Micro
- Q1: Datasheet (none) -> https://www.infineon.com/dgdl/irlml6402pbf.pdf?fileId=5546d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; Description (none) -> MOSFET MOSFT P-Ch -3.7A 65mOhm 8nC Log Lvl; Footprint (none) -> Package_TO_SOT_SMD:SOT-23; MFR (none) -> Infineon; MPN (none) -> RLML6402TRPBF; SPN (none) -> 942-IRLML6402TRPBF; SPR (none) -> Mouser; SPURL (none) -> https://www.mouser.com/ProductDetail/Infineon-Technologies/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; Value (none) -> IRLML6402
- R1: Datasheet (none) -> https://www.mouser.com/datasheet/2/54/hpreztr-777398.pdf; Description (none) -> Thick Film Resistors - SMD 1K OHM 1%; Footprint (none) -> Resistor_SMD:R_0603_1608Metric_Pad1.05x0.95mm_HandSolder; MFR (none) -> Bourns; MPN (none) -> CR0603-FX-1001ELF; SPN (none) -> 652-CR0603FX-1001ELF; SPR (none) -> Mouser; SPURL (none) -> https://www.mouser.com/ProductDetail/Bourns/CR0603-FX-1001E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; Value (none) -> 1K
- R10, R11, R12, R13, R14, R15, R2, R3, R4, R9: Datasheet (none) -> https://www.mouser.com/datasheet/2/54/hpreztr-777398.pdf; Description (none) -> Thick Film Resistors - SMD 10K OHM 1%; Footprint (none) -> Resistor_SMD:R_0603_1608Metric_Pad1.05x0.95mm_HandSolder; MFR (none) -> Bourns; MPN (none) -> CR0603-FX-1002ELF; SPN (none) -> 652-CR0603FX-1002ELF; SPR (none) -> Mouser; SPURL (none) -> https://www.mouser.com/ProductDetail/Bourns/CR0603-FX-1002E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; Value (none) -> 10K
- R16: Datasheet (none) -> https://www.mouser.com/datasheet/2/54/hpreztr-777398.pdf; Description Thick Film Resistors - SMD 1M OHM 5% -> Thick Film Resistors - SMD 1M OHM 1%; Footprint (none) -> Resistor_SMD:R_0603_1608Metric_Pad1.05x0.95mm_HandSolder; MFR Yageo -> Bourns; MPN RC0603JR-071ML -> CR0603-FX-1004ELF; SPN 603-RC0603JR-071ML -> 652-CR0603FX-1004ELF; Value (none) -> 1M
- R18: Datasheet (none) -> https://www.mouser.com/datasheet/2/54/hpreztr-777398.pdf; Description Thick Film Resistors - SMD 10K 1% 1/10W -> Thick Film Resistors - SMD 360R 1%; Footprint (none) -> Resistor_SMD:R_0603_1608Metric_Pad1.05x0.95mm_HandSolder; MFR (none) -> Bourns; MPN CR0603-FX-1002ELF -> CR0603-FX-3600ELF; SPN (none) -> 652-CR0603FX-3600ELF; SPR (none) -> Mouser; SPURL (none) -> https://www.mouser.com/ProductDetail/Bourns/CR0603-FX-3600E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; Value (none) -> 360R
- R5, R7: Datasheet (none) -> https://www.mouser.com/datasheet/2/54/hpreztr-777398.pdf; Description (none) -> Thick Film Resistors - SMD 100R OHM 1%; Footprint (none) -> Resistor_SMD:R_0603_1608Metric_Pad1.05x0.95mm_HandSolder; MFR (none) -> Bourns; MPN (none) -> CR0603-FX-1000ELF; SPN (none) -> 652-CR0603FX-1000ELF; SPR (none) -> Mouser; SPURL (none) -> https://www.mouser.com/ProductDetail/Bourns/CR0603-FX-1000E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; Value (none) -> 100R
- R6, R8: Datasheet (none) -> https://www.mouser.com/datasheet/2/54/hpreztr-777398.pdf; Description (none) -> Thick Film Resistors - SMD 360R 1%; Footprint (none) -> Resistor_SMD:R_0603_1608Metric_Pad1.05x0.95mm_HandSolder; MFR (none) -> Bourns; MPN (none) -> CR0603-FX-3600ELF; SPN (none) -> 652-CR0603FX-3600ELF; SPR (none) -> Mouser; SPURL (none) -> https://www.mouser.com/ProductDetail/Bourns/CR0603-FX-3600E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; Value (none) -> 360R
- SW1: Description (none) -> Tactile Switches 3.9x2.9x2.0mm 160gf Packaging Temp 80oC; Footprint (none) -> Button_Switch_SMD:SW_Push_SPST_NO_Alps_SKRK; MFR (none) -> ALPS; MPN (none) -> SKRKAEE020; SPN (none) -> 688-SKRKAEE020; SPR (none) -> Mouser; SPURL (none) -> https://www.mouser.com/ProductDetail/688-SKRKAEE020; Value (none) -> Reset
- SW2: Description (none) -> Tactile Switches 3.9x2.9x2.0mm 160gf Packaging Temp 80oC; Footprint (none) -> Button_Switch_SMD:SW_Push_SPST_NO_Alps_SKRK; MFR (none) -> ALPS; MPN (none) -> SKRKAEE020; SPN (none) -> 688-SKRKAEE020; SPR (none) -> Mouser; SPURL (none) -> https://www.mouser.com/ProductDetail/688-SKRKAEE020; Value (none) -> User
- SW3: footprint Button_Switch_SMD:SW_DIP_SPSTx06_Slide_Omron_A6H-6101_W6.15mm_P1.27mm -> Button_Switch_SMD:SW_DIP_SPSTx04_Slide_KingTek_DSHP04TS_W7.62mm_P1.27mm; symbol max_breakout-rescue:SW_DIP_x06-Switch -> Switch:SW_DIP_x04; Datasheet (none) -> https://www.mouser.com/datasheet/2/307/en-a6h-1221378.pdf; Footprint (none) -> Button_Switch_SMD:SW_DIP_SPSTx04_Slide_KingTek_DSHP04TS_W7.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; SPR (none) -> Mouser; Value (none) -> User DIP Switch
- U1: Datasheet (none) -> http://www.zlgmcu.com/Sipex/LDO/PDF/spx2920.pdf; Description (none) -> LDO Voltage Regulators LDO CMOS LowCurr SOT23 T&R 3K; Footprint (none) -> Package_TO_SOT_SMD:SOT-23; MFR (none) -> Diodes Inc; MPN (none) -> AP7381-33SA-7; SPN (none) -> 621-AP7381-33SA-7; SPR (none) -> Mouser; SPURL (none) -> https://www.mouser.com/ProductDetail/Diodes-Incorporated/AP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; Value (none) -> AP7381-33SA
- U2: Datasheet (none) -> https://media.digikey.com/pdf/Data%20Sheets/Intel%20PDFs/MA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; Description (none) -> CPLD 32MC 10NS 44TQFP; Footprint (none) -> Package_QFP:TQFP-44_10x10mm_P0.8mm_ThermalVias; MFR (none) -> Intel; MPN (none) -> EPM7032STC44-10FN; Value (none) -> EPM7032STC44
- U3: Datasheet (none) -> https://www.mouser.com/datasheet/2/256/maxim%20integrated%2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; Description (none) -> Supervisory Circuits 5V EconoReset w/Pushbutton; Footprint (none) -> Package_TO_SOT_SMD:SOT-23; MFR (none) -> Maxim; MPN (none) -> DS1813R-5+T&R; SPN (none) -> 700-DS1813R-5T&R; SPR (none) -> Mouser; SPURL (none) -> https://www.mouser.com/ProductDetail/Maxim-Integrated/DS181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; Value (none) -> DS1813R-5+T&R
- U4, U5: Datasheet (none) -> https://www.mouser.com/datasheet/2/256/MAX40200-1112995.pdf; Description (none) -> Supervisory Circuits Current Sense/Ideal Diode; Footprint (none) -> Package_TO_SOT_SMD:SOT-23-5_HandSoldering; MFR (none) -> Maxim; MPN (none) -> MAX40200AUK+T; SPN (none) -> 700-MAX40200AUK+T; SPR (none) -> Mouser; SPURL (none) -> https://www.mouser.com/ProductDetail/Maxim-Integrated/MAX40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; Value (none) -> MAX40200AUK
- X1: Datasheet (none) -> https://www.mouser.com/datasheet/2/96/008-0250-0-786318.pdf; Description (none) -> 50Mhz Clock Oscillator, 3.3V, HCMOS,TTL; Footprint (none) -> Oscillator:Oscillator_SMD_TXC_7C-4Pin_5.0x3.2mm_HandSolderi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; MFR (none) -> CTS; MPN (none) -> 636L3C050M00000; SPN (none) -> 774-636L3C050M00000; SPR (none) -> Mouser; SPURL (none) -> https://www.mouser.com/ProductDetail/CTS-Electronic-Compone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; Value (none) -> CTX-636 50mhz
Connections:
- net labels added: BLU, CLK, GRN, PB1, RED
- net labels removed: CLK1, LED_ENA, ~OE1
- wire segments 238 -> 230
- no-connect marks 4 -> 7
Other:
- moved on the sheet: C1, C12, C7, R10, R11, R12, R13, R18, R5, R9, SW1, SW2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
