File: max_breakout.sch (KiCad schematic (older format))
At the start: 48 parts, among them J1 Left, J2 Right, J3 AVR-JTAG-10, J4 USB_B_Micro, Q1 IRLML6402, SW1 Reset, SW2 User, SW3 User DIP Switch, SW4 ENA Switch, U1 AP7381-33SA, U2 EPM7032STC44, U3 DS1813R-5+T&R, U4 MAX40200AUK, U5 MAX40200AUK, U6 74HCT244, X1 CTX-636 50mhz

Commit message: Fixed up library references
Parts:
- C1, C10, C11, C12, C2, C3, C4, C5, C7, C8, C9: symbol max_breakout-rescue:C_Small-Device -> Device:C_Small
- C13: symbol max_breakout-rescue:C-Device -> Device:C_Small
- D1, D2: symbol max_breakout-rescue:LED-Device -> Device:LED
- R1, R10, R11, R12, R13, R14, R15, R2, R3, R4, R5, R6, R7, R8, R9: symbol max_breakout-rescue:R_Small-Device -> Device:R_Small
- R16: symbol max_breakout-rescue:R-Device -> Device:R_Small
Connections:
- wire segments 230 -> 234
Changed lines of the file:
@@
 $EndDescr
 $Comp
-L max_breakout-rescue:GND-power #PWR017
+L power:GND #PWR017
 U 1 1 5D617CA8
 P 9800 3850
@@
 $EndComp
 $Comp
-L max_breakout-rescue:C_Small-Device C?
+L Device:C_Small C?
 U 1 1 5D700E67
 P 9600 3700
@@
 $EndComp
 $Comp
-L max_breakout-rescue:C_Small-Device C?
+L Device:C_Small C?
 U 1 1 5D7A2EE6
 P 9800 3700
@@
 $EndComp
 $Comp
-L max_breakout-rescue:C_Small-Device C?
+L Device:C_Small C?
 U 1 1 5D7A2EF2
 P 10000 3700
@@
 $EndComp
 $Comp
-L max_breakout-rescue:GND-power #PWR010
+L power:GND #PWR010
 U 1 1 5D1C7065
 P 6550 2650
@@
 $EndComp
 $Comp
-L max_breakout-rescue:GND-power #PWR03
+L power:GND #PWR03
 U 1 1 5D1C706B
 P 7000 1150
@@
 $EndComp
 $Comp
-L max_breakout-rescue:R_Small-Device R?
+L Device:R_Small R?
 U 1 1 5D1C7095
 P 7250 1500
@@
 $EndComp
 $Comp
-L max_breakout-rescue:R_Small-Device R10
+L Device:R_Small R10
 U 1 1 6040DBE3
 P 4050 5100
@@
 $EndComp
 $Comp
-L max_breakout-rescue:R_Small-Device R11
+L Device:R_Small R11
 U 1 1 6040DBE9
 P 4150 5100
@@
 $EndComp
 $Comp
-L max_breakout-rescue:R_Small-Device R12
+L Device:R_Small R12
 U 1 1 6040DBEF
 P 4250 5100
@@
 $EndComp
 $Comp
-L max_breakout-rescue:R_Small-Device R13
+L Device:R_Small R13
 U 1 1 6040DBF5
 P 4350 5100
@@
 $EndComp
 $Comp
-L max_breakout-rescue:C-Device C13
+L Device:C_Small C13
 U 1 1 5CFAD747
 P 7100 5850
@@
 $EndComp
 $Comp
-L max_breakout-rescue:LED-Device D1
+L Device:LED D1
 U 1 1 5D74CDCC
 P 10850 6000
@@
 $EndComp
 $Comp
-L max_breakout-rescue:GND-power #PWR07
+L power:GND #PWR07
 U 1 1 5D838E8D
 P 2200 2250
@@
 $EndComp
 $Comp
-L max_breakout-rescue:R_Small-Device R?
+L Device:R_Small R?
 U 1 1 5D350372
 P 7350 1500
@@
 $EndComp
 $Comp
-L max_breakout-rescue:R_Small-Device R?
+L Device:R_Small R?
 U 1 1 5D351229
 P 7450 1500
@@
 $EndComp
 $Comp
-L max_breakout-rescue:R_Small-Device R?
+L Device:R_Small R?
 U 1 1 5D351612
 P 7550 1500
@@
 $EndComp
 $Comp
-L max_breakout-rescue:C_Small-Device C?
+L Device:C_Small C?
 U 1 1 5D39812A
 P 1900 2150
@@
 $EndComp
 $Comp
-L max_breakout-rescue:GND-power #PWR012
+L power:GND #PWR012
 U 1 1 5D42A074
 P 10850 6150
@@
 $EndComp
 $Comp
-L max_breakout-rescue:R_Small-Device R?
+L Device:R_Small R?
 U 1 1 5D74F407
 P 10850 5750
@@
 $EndComp
 $Comp
-L max_breakout-rescue:GND-power #PWR032
+L power:GND #PWR032
 U 1 1 5D4C5742
 P 3100 5650
@@
 $EndComp
 $Comp
-L max_breakout-rescue:R_Small-Device R?
+L Device:R_Small R?
 U 1 1 5D3835DF
 P 2900 1900
@@
 $EndComp
 $Comp
-L max_breakout-rescue:LED-Device D2
+L Device:LED D2
 U 1 1 5D403063
 P 7750 3200
@@
 $EndComp
 $Comp
-L max_breakout-rescue:GND-power #PWR014
+L power:GND #PWR014
 U 1 1 5D403069
 P 7750 3600
@@
 $EndComp
 $Comp
-L max_breakout-rescue:R_Small-Device R?
+L Device:R_Small R?
 U 1 1 5D47E16C
 P 7750 3450
@@
 $EndComp
 $Comp
-L max_breakout-rescue:GND-power #PWR028
+L power:GND #PWR028
 U 1 1 5D385EAD
 P 9650 5550
@@
 $EndComp
 $Comp
-L max_breakout-rescue:GND-power #PWR027
+L power:GND #PWR027
 U 1 1 5D38472E
 P 8300 5550
@@
 $EndComp
 $Comp
-L max_breakout-rescue:C_Small-Device C?
+L Device:C_Small C?
 U 1 1 5DA6A045
 P 10350 5200
@@
 $EndComp
 $Comp
-L max_breakout-rescue:C_Small-Device C?
+L Device:C_Small C?
 U 1 1 5D39F958
 P 7450 5200
@@
 $EndComp
 $Comp
-L max_breakout-rescue:C_Small-Device C?
+L Device:C_Small C?
 U 1 1 5D3A29B6
 P 9100 5250
@@
 $EndComp
 $Comp
-L max_breakout-rescue:GND-power #PWR024
+L power:GND #PWR024
 U 1 1 5D3A29B7
 P 9100 5350
@@
 $EndComp
 $Comp
-L max_breakout-rescue:GND-power #PWR023
+L power:GND #PWR023
 U 1 1 5D3A31C4
 P 8850 5350
@@
 $EndComp
 $Comp
-L max_breakout-rescue:GND-power #PWR025
+L power:GND #PWR025
 U 1 1 5D47C55F
 P 10350 5350
@@
 $EndComp
 $Comp
-L max_breakout-rescue:C_Small-Device C?
+L Device:C_Small C?
 U 1 1 5D480F38
 P 8850 5250
@@
 $EndComp
 $Comp
-L max_breakout-rescue:GND-power #PWR022
+L power:GND #PWR022
 U 1 1 5D39F959
 P 7450 5300
@@
 $EndComp
 $Comp
-L max_breakout-rescue:R-Device R?
+L Device:R_Small R?
 U 1 1 5CFB0AB4
 P 6900 5850
@@
 $EndComp
 $Comp
-L max_breakout-rescue:GND-power #PWR031
+L power:GND #PWR031
 U 1 1 5D486EFD
 P 7300 6150
@@
 $EndComp
 $Comp
-L max_breakout-rescue:R_Small-Device R?
+L Device:R_Small R?
 U 1 1 5D42FF74
 P 7350 2850
@@
 $EndComp
 $Comp
-L max_breakout-rescue:C_Small-Device C?
+L Device:C_Small C?
 U 1 1 5D3C4E3F
 P 10200 3700
@@
 $EndComp
 $Comp
-L max_breakout-rescue:C_Small-Device C?
+L Device:C_Small C?
 U 1 1 5D44D976
 P 9400 3700
@@
 $EndComp
 $Comp
-L max_breakout-rescue:GND-power #PWR06
+L power:GND #PWR06
 U 1 1 5D3EE1AD
 P 1400 1800
@@
 $EndComp
 $Comp
-L max_breakout-rescue:GND-power #PWR015
+L power:GND #PWR015
 U 1 1 5D46649B
 P 4550 3800
@@
 $EndComp
 $Comp
-L max_breakout-rescue:GND-power #PWR013
+L power:GND #PWR013
 U 1 1 5D3F5930
 P 1300 3750
@@
 $EndComp
 $Comp
-L max_breakout-rescue:R_Small-Device R9
+L Device:R_Small R9
 U 1 1 5D436631
 P 3100 6400
@@
 $EndComp
 $Comp
-L max_breakout-rescue:C_Small-Device C?
+L Device:C_Small C?
 U 1 1 5D437E32
 P 3100 6750
@@
 $EndComp
 $Comp
-L max_breakout-rescue:GND-power #PWR029
+L power:GND #PWR029
 U 1 1 5D43846A
 P 2650 7000
@@
 $EndComp
 $Comp
-L max_breakout-rescue:GND-power #PWR030
+L power:GND #PWR030
 U 1 1 5D438687
 P 3100 7000
@@
 $EndComp
 $Comp
-L max_breakout-rescue:R_Small-Device R14
+L Device:R_Small R14
 U 1 1 5D98B205
 P 4350 6900
@@
 $EndComp
 $Comp
-L max_breakout-rescue:R_Small-Device R15
+L Device:R_Small R15
 U 1 1 5D98B20B
 P 4450 6900
@@
 $EndComp
 $Comp
-L max_breakout-rescue:GND-power #PWR034
+L power:GND #PWR034
 U 1 1 5DF28657
 P 4500 6150
@@
 $EndComp
 $Comp
-L max_breakout-rescue:GND-power #PWR036
+L power:GND #PWR036
 U 1 1 5DFDF18A
 P 5000 6750
@@
 	7300 5500 7300 6000
 Wire Wire Line
-	7300 6000 7100 6000
-Wire Wire Line
 	10350 5300 10350 5350
 Wire Wire Line
@@
 	700  4550 6424 4550
 Wire Wire Line
-	6900 6000 7100 6000
-Wire Wire Line
 	7000 5700 7100 5700
 Wire Wire Line
@@
 Connection ~ 10350 5100
 Connection ~ 7450 5100
-Connection ~ 6900 5700
 Connection ~ 4500 3700
 Connection ~ 4600 3700
@@
 Connection ~ 3100 6550
 Connection ~ 1300 3650
-Connection ~ 7100 6000
 Connection ~ 7000 5700
 Connection ~ 3350 5550
@@
 NoConn ~ 3350 6650
 NoConn ~ 3950 6650
+Wire Wire Line
+	6900 6000 7100 6000
+Wire Wire Line
+	6900 5750 6900 5700
+Connection ~ 6900 5700
+Wire Wire Line
+	6900 5950 6900 6000
+Wire Wire Line
+	7100 5950 7100 6000
+Connection ~ 7100 6000
+Wire Wire Line
+	7100 6000 7300 6000
+Wire Wire Line
+	7100 5750 7100 5700
 $EndSCHEMATC
