File: max_breakout.sch (KiCad schematic (older format))
At the start: 53 parts, among them J1 USB_B_Micro, J2 AVR-JTAG-10, J3 Left, J4 Right, SW1 User, SW2 User, U1 MAX40203AUK+T, U2 74HCT1G04, U3 EPM7032STC44, U4 LP2985-5.0, U5 LP2985-3.3, U6 74HCT125, X1 CTX-636 50mhz

Commit message: added open-drain clock driver, pull-ups for JTAG, removed TDI led
Parts:
- removed D1: Green, LED_SMD:LED_0603_1608Metric_Pad1.05x0.95mm_HandSolder, symbol Device:LED
- removed R1: 1K, Resistor_SMD:R_0603_1608Metric_Pad1.05x0.95mm_HandSolder, symbol Device:R_Small
- removed U2: 74HCT1G04, Package_TO_SOT_SMD:SOT-353_SC-70-5, symbol 74xGxx:74LVC1G04
- added R4: 10K, Resistor_SMD:R_0603_1608Metric_Pad1.05x0.95mm_HandSolder, symbol Device:R_Small
- added U5: 74LVC1G38, Package_SO:TSOP-5_1.65x3.05mm_P0.95mm, symbol 74xGxx:74LVC1G38
- R5: value 33R -> 10K; Description Thick Film Resistors - SMD 100R OHM 1% -> Thick Film Resistors - SMD 10K OHM 1%; MPN CR0603-FX-1000ELF -> CR0603-FX-1002ELF; SPN 652-CR0603FX-1000ELF -> 652-CR0603FX-1002ELF; SPURL https://www.mouser.com/ProductDetail/Bourns/CR0603-FX-1000E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 -> https://www.mouser.com/ProductDetail/Bourns/CR0603-FX-1002E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
- renumbered C13 to C12, C14 to C13, C15 to C14, C16 to C15, C17 to C16, C12 to C17, R9 to R11, R13 to R12, R12 to R13, R15 to R14, R14 to R15, R11 to R16, R4 to R6, R6 to R7, R7 to R8, R8 to R9, U5 to U6, U6 to U7
Connections:
- wire segments 213 -> 222
Other:
- note removed: "JTAG Activity"
- moved on the sheet: C17, C18, C7, J2, JP1, R11, R13, R16, R6, R7, R8, R9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

Commit message: fixed layout of regulators
Parts:
- C1: value .33uF -> 1uF
- C10, C5: value 10nF -> 100nF
- C11, C6: value 100uF -> 2.2uF; footprint Capacitor_SMD:C_1206_3216Metric_Pad1.42x1.75mm_HandSolder -> Capacitor_SMD:C_0603_1608Metric_Pad1.05x0.95mm_HandSolder
Changed lines of the file:
@@
 AR Path="/5D39F958" Ref="C1"  Part="1"
 F 0 "C1" H 1892 1146 50  0000 L CNN
-F 1 ".33uF" H 1892 1055 32  0000 L CNN
+F 1 "1uF" H 1892 1055 32  0000 L CNN
 F 2 "Capacitor_SMD:C_0603_1608Metric_Pad1.05x0.95mm_HandSolder" H 1800 1100 50  0001 C CNN
 F 3 "https://www.mouser.com/datasheet/2/396/mlcc02_e-1307760.pdf" H 1800 1100 50  0001 C CNN
@@
 	9700 4950 9400 4950
 Wire Wire Line
-	9700 6050 9400 6050
+	9700 6250 9400 6250
 Wire Wire Line
 	9700 5050 9400 5050
@@
 $EndComp
 Wire Wire Line
-	9700 6150 9400 6150
+	9700 6050 9400 6050
 Wire Wire Line
 	900  1600 900  1550
@@
 Text GLabel 3450 950  2    50   Output ~ 0
 Vin
-Text GLabel 9400 6050 0    50   Input ~ 0
+Text GLabel 9400 6250 0    50   Input ~ 0
 Vin
-Text GLabel 9400 6150 0    50   Output ~ 0
+Text GLabel 9400 6050 0    50   Output ~ 0
 5V
 Text GLabel 8100 6150 0    50   Output ~ 0
@@
 P 3000 3450
 F 0 "C11" H 3100 3500 50  0000 L CNN
-F 1 "100uF" H 3100 3400 50  0000 L CNN
-F 2 "Capacitor_SMD:C_1206_3216Metric_Pad1.42x1.75mm_HandSolder" H 3000 3450 50  0001 C CNN
+F 1 "2.2uF" H 3100 3400 50  0000 L CNN
+F 2 "Capacitor_SMD:C_0603_1608Metric_Pad1.05x0.95mm_HandSolder" H 3000 3450 50  0001 C CNN
 F 3 "~" H 3000 3450 50  0001 C CNN
 	1    3000 3450
@@
 P 2200 3450
 F 0 "C10" H 2292 3496 50  0000 L CNN
-F 1 "10nF" H 2292 3405 50  0000 L CNN
+F 1 "100nF" H 2292 3405 50  0000 L CNN
 F 2 "Capacitor_SMD:C_0603_1608Metric_Pad1.05x0.95mm_HandSolder" H 2200 3450 50  0001 C CNN
 F 3 "~" H 2200 3450 50  0001 C CNN
@@
 P 3000 2550
 F 0 "C6" H 3100 2600 50  0000 L CNN
-F 1 "100uF" H 3100 2500 50  0000 L CNN
-F 2 "Capacitor_SMD:C_1206_3216Metric_Pad1.42x1.75mm_HandSolder" H 3000 2550 50  0001 C CNN
+F 1 "2.2uF" H 3100 2500 50  0000 L CNN
+F 2 "Capacitor_SMD:C_0603_1608Metric_Pad1.05x0.95mm_HandSolder" H 3000 2550 50  0001 C CNN
 F 3 "~" H 3000 2550 50  0001 C CNN
 	1    3000 2550
@@
 P 2200 2550
 F 0 "C5" H 2292 2596 50  0000 L CNN
-F 1 "10nF" H 2292 2505 50  0000 L CNN
+F 1 "100nF" H 2292 2505 50  0000 L CNN
 F 2 "Capacitor_SMD:C_0603_1608Metric_Pad1.05x0.95mm_HandSolder" H 2200 2550 50  0001 C CNN
 F 3 "~" H 2200 2550 50  0001 C CNN
@@
 Text Label 9500 4950 0    50   ~ 0
 CLK
-Text Label 9550 6250 0    50   ~ 0
+Text Label 9550 6150 0    50   ~ 0
 GND
 Wire Wire Line
-	9700 6250 9250 6250
+	9700 6150 9050 6150
 $Comp
 L power:GND #PWR031
 U 1 1 5F0609D2
-P 9250 6250
+P 9050 6150
 AR Path="/5F0609D2" Ref="#PWR031"  Part="1"
 AR Path="/5D0F9837/5F0609D2" Ref="#PWR?"  Part="1"
@@
 AR Path="/5CFABACD/5CFFC458/5F0609D2" Ref="#PWR?"  Part="1"
 AR Path="/5D65A6A0/5F0609D2" Ref="#PWR?"  Part="1"
-F 0 "#PWR031" H 9250 6000 50  0001 C CNN
-F 1 "GND" H 9255 6077 50  0000 C CNN
-F 2 "" H 9250 6250 50  0001 C CNN
-F 3 "" H 9250 6250 50  0001 C CNN
-	1    9250 6250
-	1    0    0    -1
-$EndComp
+F 0 "#PWR031" H 9050 5900 50  0001 C CNN
+F 1 "GND" H 9055 5977 50  0000 C CNN
+F 2 "" H 9050 6150 50  0001 C CNN
+F 3 "" H 9050 6150 50  0001 C CNN
+	1    9050 6150
+	1    0    0    -1
+$EndComp

Commit message: added level shifter on clock
Parts:
- added R17: 10K, Resistor_SMD:R_0603_1608Metric_Pad1.05x0.95mm_HandSolder, symbol Device:R_Small
Connections:
- wire segments 222 -> 224
Changed lines of the file:
@@
 Text Notes 700  4450 0    50   ~ 0
 USER GPIO
-Text Notes 5450 2550 0    50   ~ 0
+Text Notes 5300 2550 0    50   ~ 0
 50Mhz Clock
 Text Notes 10050 2550 2    50   ~ 0
@@
 	5400 2950 5400 3000
 Wire Wire Line
-	5950 2950 6850 2950
+	5950 2950 6100 2950
+$Comp
+L Device:R_Small R?
+U 1 1 5EB86C95
+P 6100 2600
+AR Path="/5D0F9837/5EB86C95" Ref="R?"  Part="1"
+AR Path="/5CFABACD/5D0BF766/5EB86C95" Ref="R?"  Part="1"
+AR Path="/5D1AF052/5EB86C95" Ref="R?"  Part="1"
+AR Path="/5EB86C95" Ref="R17"  Part="1"
+F 0 "R17" H 6150 2600 50  0000 L CNN
+F 1 "10K" V 6100 2550 32  0000 L CNN
+F 2 "Resistor_SMD:R_0603_1608Metric_Pad1.05x0.95mm_HandSolder" H 6100 2600 50  0001 C CNN
+F 3 "https://www.mouser.com/datasheet/2/54/hpreztr-777398.pdf" H 6100 2600 50  0001 C CNN
+F 4 "Thick Film Resistors - SMD 10K OHM 1%" H 6100 2800 50  0001 C CNN "Description"
+F 5 "Bourns" H 6100 2800 50  0001 C CNN "MFR"
+F 6 "CR0603-FX-1002ELF" H 6100 2800 50  0001 C CNN "MPN"
+F 7 "652-CR0603FX-1002ELF" H 6100 2800 50  0001 C CNN "SPN"
+F 8 "Mouser" H 6100 2800 50  0001 C CNN "SPR"
+F 9 "https://www.mouser.com/ProductDetail/Bourns/CR0603-FX-1002ELF?qs=%2Fha2pyFadugVmr2gairtN7QOhA7v8%2FIyn%2F6JFX3D8auJGt%2FYJ41PlQ%3D%3D" H 6100 2800 50  0001 C CNN "SPURL"
+	1    6100 2600
+	-1   0    0    -1
+$EndComp
+$Comp
+L power:VCC #PWR037
+U 1 1 5EB86C9B
+P 6100 2500
+F 0 "#PWR037" H 6100 2350 50  0001 C CNN
+F 1 "VCC" H 6117 2673 50  0000 C CNN
+F 2 "" H 6100 2500 50  0001 C CNN
+F 3 "" H 6100 2500 50  0001 C CNN
+	1    6100 2500
+	1    0    0    -1
+$EndComp
+Wire Wire Line
+	6100 2700 6100 2950
+Connection ~ 6100 2950
+Wire Wire Line
+	6100 2950 6850 2950
 $EndSCHEMATC

Commit message: removed extraneous pullups
Parts:
- removed R17, R4, R5: 10K, Resistor_SMD:R_0603_1608Metric_Pad1.05x0.95mm_HandSolder, symbol Device:R_Small
- removed R7, R8: 1K, Resistor_SMD:R_0603_1608Metric_Pad1.05x0.95mm_HandSolder, symbol Device:R_Small
- removed U5: 74LVC1G38, Package_SO:TSOP-5_1.65x3.05mm_P0.95mm, symbol 74xGxx:74LVC1G38
- C10, C5: value 100nF -> 10nF
- renumbered D2 to D1, D3 to D2, D4 to D3, D5 to D4, D6 to D5, R2 to R1, R13 to R10, R14 to R11, R15 to R12, R16 to R13, R3 to R2, R6 to R3, R9 to R6, R10 to R7, R11 to R8, R12 to R9, U3 to U2, U4 to U3, U6 to U4, U7 to U5
Connections:
- net labels added: GCLRn, OE1
- wire segments 224 -> 204
Other:
- moved on the sheet: C8, X1

Commit message: rewired pushbuttons to input pins
Parts:
- added JP2: clk ena, Connector_PinHeader_2.54mm:PinHeader_1x02_P2.54mm_Vertical, symbol Device:Jumper_NO_Small
- renumbered C3 to C1, C11 to C10, C2 to C11, C8 to C12, C12 to C13, C13 to C14, C14 to C15, C15 to C16, C16 to C17, C7 to C18, C4 to C2, C9 to C3, C17 to C4, C18 to C5, C1 to C6, C5 to C7, C10 to C8, C6 to C9, J3 to J2, J4 to J3, J2 to J4, R3 to R10, R6 to R11, R8 to R2, R13 to R3, R10 to R4, R2 to R5, R7 to R6, R9 to R7, R11 to R8, R12 to R9, U3 to U1, U4 to U2, U1 to U3, U5 to U4, U2 to U5
Connections:
- net labels added: B18, B32
- wire segments 204 -> 205

Commit message: switches push buttons and leds to active high, silk screen enhancements
Parts:
- removed C4, C5: 10nF, Capacitor_SMD:C_0603_1608Metric_Pad1.05x0.95mm_HandSolder, symbol Device:C_Small
- added R12, R7: 10K, Resistor_SMD:R_0603_1608Metric_Pad1.05x0.95mm_HandSolder, symbol Device:R_Small
- renumbered C6 to C1, C8 to C10, C10 to C11, C13 to C12, C14 to C13, C15 to C14, C16 to C15, C17 to C16, C11 to C2, C1 to C3, C2 to C4, C7 to C5, C9 to C6, C18 to C7, C12 to C8, C3 to C9, J4 to J2, J2 to J3, J3 to J4, JP2 to JP1, JP1 to JP2, R4 to R10, R9 to R11, R3 to R13, R5 to R2, R10 to R3, R11 to R4, R6 to R5, R7 to R6, R2 to R8, R8 to R9, U3 to U1, U5 to U2, U1 to U3, U2 to U4, U4 to U5
Connections:
- wire segments 205 -> 207
Other:
- moved on the sheet: D2, D3, D4, D5, JP2, R10, R13, R8, SW1, SW2

Commit message: schematic cleanup
Parts:
- removed R12, R13, R8: 10K, Resistor_SMD:R_0603_1608Metric_Pad1.05x0.95mm_HandSolder, symbol Device:R_Small
- added R10, R11, R9: 10K, Resistor_SMD:R_0603_1608Metric_Pad1.05x0.95mm_HandSolder, symbol Device:R_Small
- renumbered R11 to R12, R10 to R13, R9 to R8
Connections:
- wire segments 207 -> 211
Other:
- moved on the sheet: JP2, R13

Commit message: made USB shield a NC, add nofill region around xtal
Parts:
- removed C3: 100nF, Capacitor_SMD:C_0603_1608Metric_Pad1.05x0.95mm_HandSolder, symbol Device:C_Small
- removed R1: 1M, Resistor_SMD:R_0603_1608Metric_Pad1.05x0.95mm_HandSolder, symbol Device:R_Small
- renumbered C4 to C1, C12 to C10, C13 to C11, C14 to C12, C15 to C13, C16 to C14, C7 to C15, C9 to C2, C1 to C3, C5 to C4, C10 to C5, C2 to C6, C6 to C7, C11 to C8, C8 to C9, J3 to J2, J4 to J3, J2 to J4, JP2 to JP1, JP1 to JP2, R10 to R1, R12 to R10, R3 to R11, R4 to R12, R11 to R2, R7 to R3, R9 to R4, R13 to R5, R2 to R6, R5 to R7, R6 to R8, R8 to R9, U3 to U1, U4 to U2, U1 to U3, U5 to U4, U2 to U5
Connections:
- wire segments 211 -> 204
- no-connect marks 5 -> 6
Other:
- moved on the sheet: C3, C6, J1, U3
